Commit message: small correction to color frame position

File: urdf/realsense-RS200.macro.xacro (robot description, xacro)
@@ -1,5 +1,5 @@
 <?xml version="1.0" ?>
 <!--Develped by Daniel Ordonez 22.05.2018 - daniels.ordonez@gmail.com
-	INFORMATION:
+	INFORMATIONd:
 		This xacro file a URDF representation of the intel real sense RS200 with the
         virtual links representing the position of:
@@ -53,4 +53,5 @@
     	<parent link="rs200_camera" />
     	<child link="depth" />
+		<origin xyz="0 -0.03 0.004" rpy="0 0 0">
  	</joint>
 	<joint name="ired1_joint" type="fixed">

Commit message: Format URDF

File: urdf/realsense-RS200.macro.xacro (robot description, xacro)
@@ -1,6 +1,6 @@
 <?xml version="1.0" ?>
 <!--Develped by Daniel Ordonez 22.05.2018 - daniels.ordonez@gmail.com
-	INFORMATIONd:
-		This xacro file a URDF representation of the intel real sense RS200 with the
+    INFORMATIONd:
+        This xacro file a URDF representation of the intel real sense RS200 with the
         virtual links representing the position of:
             * The RGB color camera
@@ -8,175 +8,175 @@
             * Infrared 2 camera
             * Virtual depth coordinate frame
-		Configured to work with Gazebo if desired.
+        Configured to work with Gazebo if desired.
 -->
 <robot xmlns:xacro="http://ros.org/wiki/xacro">
 <xacro:macro name="realsense-rs200">
-	<!-- Camera link -->
-	<link name="rs200_camera">
-		<visual>
-			<origin rpy="0 0 0" xyz="0 0 0"/>
-			<geometry>
-				<mesh filename="package://realsense_gazebo_plugin/models/realsense_camera/meshes/realsense.dae"/>
-			</geometry>
-		</visual>
-		<collision>
-			<geometry>
-          		<box size="0.0078 0.130 0.0192"/>
-        	</geometry>
-		</collision>
-		<inertial>
-        	<mass value="0.0615752"/>
-			<origin rpy="0 0 0" xyz="0 0 0"/>
-			<inertia ixx="9.108e-05"
-					 ixy="0"
-				     ixz="0"
-				     iyy="2.51e-06"
-				     iyz="0"
-				     izz="8.931e-05"
-			/>
-      	</inertial>
-	</link>
-	<!-- Virtual links representing the cameras positons and orientations-->
-	<link name="color" />
-	<link name="depth" />
-	<link name="ired1" />
-	<link name="ired2" />
-	<!-- Joints positioning the virtual links with respect to the camera main link-->
-	<joint name="color_joint" type="fixed">
-    	<parent link="rs200_camera" />
-    	<child link="color" />
-		<!--<origin xyz="0 -0.046 0.004" rpy="0 0 0"/>-->
-		<!-- The default position is change since in Rviz the cloud depth axis is Z not X-->
-		<origin xyz="0 -0.046 0.004" rpy="${pi/2} ${pi} ${pi/2}"/>
- 	</joint>
-	<joint name="depth_joint" type="fixed">
-    	<parent link="rs200_camera" />
-    	<child link="depth" />
-		<origin xyz="0 -0.03 0.004" rpy="0 0 0">
- 	</joint>
-	<joint name="ired1_joint" type="fixed">
-    	<parent link="rs200_camera" />
-    	<child link="ired1" />
-		<origin xyz="0 -0.06 0.004" rpy="0 0 0"/>
- 	</joint>
-	<joint name="ired2_joint" type="fixed">
-		<parent link="rs200_camera" />
-		<child link="ired2" />
-		<origin xyz="0 0.01 0.004" rpy="0 0 0"/>
- 	</joint>
+    <!-- Camera link -->
+    <link name="rs200_camera">
+        <visual>
+            <origin rpy="0 0 0" xyz="0 0 0"/>
+            <geometry>
+                <mesh filename="package://realsense_gazebo_plugin/models/realsense_camera/meshes/realsense.dae"/>
+            </geometry>
+        </visual>
+        <collision>
+            <geometry>
+                <box size="0.0078 0.130 0.0192"/>
+            </geometry>
+        </collision>
+        <inertial>
+            <mass value="0.0615752"/>
+            <origin rpy="0 0 0" xyz="0 0 0"/>
+            <inertia ixx="9.108e-05"
+                     ixy="0"
+                     ixz="0"
+                     iyy="2.51e-06"
+                     iyz="0"
+                     izz="8.931e-05"
+            />
+        </inertial>
+    </link>
+    <!-- Virtual links representing the cameras positons and orientations-->
+    <link name="color" />
+    <link name="depth" />
+    <link name="ired1" />
+    <link name="ired2" />
+    <!-- Joints positioning the virtual links with respect to the camera main link-->
+    <joint name="color_joint" type="fixed">
+        <parent link="rs200_camera" />
+        <child link="color" />
+        <!-- <origin xyz="0 -0.046 0.004" rpy="0 0 0"/> -->
+        <!-- The default position is change since in Rviz the cloud depth axis is Z not X-->
+        <origin xyz="0 -0.046 0.004" rpy="${pi/2} ${pi} ${pi/2}"/>
+    </joint>
+    <joint name="depth_joint" type="fixed">
+        <parent link="rs200_camera" />
+        <child link="depth" />
+        <origin xyz="0 -0.03 0.004" rpy="0 0 0"/>
+    </joint>
+    <joint name="ired1_joint" type="fixed">
+        <parent link="rs200_camera" />
+        <child link="ired1" />
+        <origin xyz="0 -0.06 0.004" rpy="0 0 0"/>
+    </joint>
+    <joint name="ired2_joint" type="fixed">
+        <parent link="rs200_camera" />
+        <child link="ired2" />
+        <origin xyz="0 0.01 0.004" rpy="0 0 0"/>
+    </joint>
 <!-- **********************************************************-->
 <!-- GAZEBO DEFINITIONS ***************************************-->
-	<!-- Load plugin to the model ("robot" in urdf format)-->
-	<gazebo>
-		<plugin name="realsense_plugin" filename="librealsense_gazebo_plugin.so"/>
-		<!--<pose frame="">0 0 0.015 0 0 0</pose>-->
-	</gazebo>
-	<!-- Load parameters to model's main link-->
-	<gazebo reference="rs200_camera">
-		<self_collide>0</self_collide>
-		<enable_wind>0</enable_wind>
-		<kinematic>0</kinematic>
-		<gravity>1</gravity>
-		<!--<mu>1</mu>-->
-		<mu2>1</mu2>
-		<fdir1>0 0 0</fdir1>
-		<!--<slip1>0</slip1>
-		<slip2>0</slip2>-->
-		<kp>1e+13</kp>
-		<kd>1</kd>
-		<!--<max_vel>0.01</max_vel>
-		<min_depth>0</min_depth>-->
-		<sensor name="color" type="camera">
-			<pose frame="">0 -0.046 0.004 0 0 0</pose>
-			<camera name="__default__">
-			<horizontal_fov>1.047</horizontal_fov>
-			<image>
-				<width>640</width>
-				<height>480</height>
-				<format>RGB_INT8</format>
-			</image>
-			<clip>
-				<near>0.1</near>
-				<far>100</far>
-			</clip>
-			<noise>
-				<type>gaussian</type>
-				<mean>0.0</mean>
-				<stddev>0.007</stddev>
-			</noise>
-			</camera>
-			<always_on>1</always_on>
-			<update_rate>60</update_rate>
-			<visualize>1</visualize>
-		</sensor>
-		<sensor name="ired1" type="camera">
-			<pose frame="">0 -0.06 0.004 0 0 0</pose>
-			<camera name="__default__">
-			<horizontal_fov>1.047</horizontal_fov>
-			<image>
-				<width>640</width>
-				<height>480</height>
-				<format>L_INT8</format>
-			</image>
-			<clip>
-				<near>0.1</near>
-				<far>100</far>
-			</clip>
-			<noise>
-				<type>gaussian</type>
-				<mean>0.0</mean>
-				<stddev>0.05</stddev>
-			</noise>
-			</camera>
-			<always_on>1</always_on>
-			<update_rate>60</update_rate>
-			<visualize>0</visualize>
-		</sensor>
-		<sensor name="ired2" type="camera">
-			<pose frame="">0 0.01 0.004 0 0 0</pose>
-			<camera name="__default__">
-			<horizontal_fov>1.047</horizontal_fov>
-			<image>
-				<width>640</width>
-				<height>480</height>
-				<format>L_INT8</format>
-			</image>
-			<clip>
-				<near>0.1</near>
-				<far>100</far>
-			</clip>
-			<noise>
-				<type>gaussian</type>
-				<mean>0.0</mean>
-				<stddev>0.05</stddev>
-			</noise>
-			</camera>
-			<always_on>1</always_on>
-			<update_rate>60</update_rate>
-			<visualize>0</visualize>
-		</sensor>
-		<sensor name="depth" type="depth">
-			<pose frame="">0 -0.03 0.004 0 0 0</pose>
-			<camera name="__default__">
-			<horizontal_fov>1.047</horizontal_fov>
-			<image>
-				<width>640</width>
-				<height>480</height>
-			</image>
-			<clip>
-				<near>0.1</near>
-				<far>100</far>
-			</clip>
-			<noise>
-				<type>gaussian</type>
-				<mean>0.0</mean>
-				<stddev>0.100</stddev>
-			</noise>
-			</camera>
-			<always_on>1</always_on>
-			<update_rate>60</update_rate>
-			<visualize>0</visualize>
-		</sensor>
-	</gazebo>
+    <!-- Load plugin to the model ("robot" in urdf format)-->
+    <gazebo>
+        <plugin name="realsense_plugin" filename="librealsense_gazebo_plugin.so"/>
+        <!--<pose frame="">0 0 0.015 0 0 0</pose>-->
+    </gazebo>
+    <!-- Load parameters to model's main link-->
+    <gazebo reference="rs200_camera">
+        <self_collide>0</self_collide>
+        <enable_wind>0</enable_wind>
+        <kinematic>0</kinematic>
+        <gravity>1</gravity>
+        <!--<mu>1</mu>-->
+        <mu2>1</mu2>
+        <fdir1>0 0 0</fdir1>
+        <!--<slip1>0</slip1>
+        <slip2>0</slip2>-->
+        <kp>1e+13</kp>
+        <kd>1</kd>
+        <!--<max_vel>0.01</max_vel>
+        <min_depth>0</min_depth>-->
+        <sensor name="color" type="camera">
+            <pose frame="">0 -0.046 0.004 0 0 0</pose>
+            <camera name="__default__">
+            <horizontal_fov>1.047</horizontal_fov>
+            <image>
+                <width>640</width>
+                <height>480</height>
+                <format>RGB_INT8</format>
+            </image>
+            <clip>
+                <near>0.1</near>
+                <far>100</far>
+            </clip>
+            <noise>
+                <type>gaussian</type>
+                <mean>0.0</mean>
+                <stddev>0.007</stddev>
+            </noise>
+            </camera>
+            <always_on>1</always_on>
+            <update_rate>60</update_rate>
+            <visualize>1</visualize>
+        </sensor>
+        <sensor name="ired1" type="camera">
+            <pose frame="">0 -0.06 0.004 0 0 0</pose>
+            <camera name="__default__">
+            <horizontal_fov>1.047</horizontal_fov>
+            <image>
+                <width>640</width>
+                <height>480</height>
+                <format>L_INT8</format>
+            </image>
+            <clip>
+                <near>0.1</near>
+                <far>100</far>
+            </clip>
+            <noise>
+                <type>gaussian</type>
+                <mean>0.0</mean>
+                <stddev>0.05</stddev>
+            </noise>
+            </camera>
+            <always_on>1</always_on>
+            <update_rate>60</update_rate>
+            <visualize>0</visualize>
+        </sensor>
+        <sensor name="ired2" type="camera">
+            <pose frame="">0 0.01 0.004 0 0 0</pose>
+            <camera name="__default__">
+            <horizontal_fov>1.047</horizontal_fov>
+            <image>
+                <width>640</width>
+                <height>480</height>
+                <format>L_INT8</format>
+            </image>
+            <clip>
+                <near>0.1</near>
+                <far>100</far>
+            </clip>
+            <noise>
+                <type>gaussian</type>
+                <mean>0.0</mean>
+                <stddev>0.05</stddev>
+            </noise>
+            </camera>
+            <always_on>1</always_on>
+            <update_rate>60</update_rate>
+            <visualize>0</visualize>
+        </sensor>
+        <sensor name="depth" type="depth">
+            <pose frame="">0 -0.03 0.004 0 0 0</pose>
+            <camera name="__default__">
+            <horizontal_fov>1.047</horizontal_fov>
+            <image>
+                    <width>640</width>
+                    <height>480</height>
+            </image>
+            <clip>
+                    <near>0.1</near>
+                    <far>100</far>
+            </clip>
+            <noise>
+                    <type>gaussian</type>
+                    <mean>0.0</mean>
+                    <stddev>0.100</stddev>
+            </noise>
+            </camera>
+            <always_on>1</always_on>
+            <update_rate>60</update_rate>
+            <visualize>0</visualize>
+        </sensor>
+    </gazebo>
 </xacro:macro>
 </robot>

File: urdf/rs200_simulation.xacro (robot description, xacro)
@@ -1,19 +1,19 @@
 <?xml version="1.0"?>
 <!--Develped by Daniel Ordonez 22.05.2018 - daniels.ordonez@gmail.com
-	INFORMATION:
-		This is an example of how to use the realsense-rs200 macro function.
+  INFORMATION:
+    This is an example of how to use the realsense-rs200 macro function.
 -->
 <robot name="robot_with_rs200" xmlns:xacro="http://ros.org/wiki/xacro">
-  <!-- Import macro for realsense-RS200 camera-->
-  <xacro:include filename="$(find robot_eyes)/urdf/realsense-RS200.macro.xacro" />
-  <!-- Create camera instance -->
-  <xacro:realsense-rs200 />
-  <!-- Gazebo world link required to position the robot with respect to origin-->
-  <link name="world"/>
-  <!-- Place camera referenced to world frame-->
-  <joint name="realsense_joint" type="fixed">
-    <parent link="world" />
-    <child link="rs200_camera" />
-    <origin xyz="0 0 1.0" rpy="0 0 0"/>
-  </joint>
+    <!-- Import macro for realsense-RS200 camera-->
+    <xacro:include filename="$(find realsense_gazebo_plugin)/urdf/realsense-RS200.macro.xacro"/>
+    <!-- Create camera instance -->
+    <xacro:realsense-rs200/>
+    <!-- Gazebo world link required to position the robot with respect to origin-->
+    <link name="world"/>
+    <!-- Place camera referenced to world frame-->
+    <joint name="realsense_joint" type="fixed">
+        <parent link="world"/>
+        <child link="rs200_camera"/>
+        <origin rpy="0 0 0" xyz="0 0 1.0"/>
+    </joint>
 </robot>

Commit message: Add prefix and parent to RS200 macro
This allows the use of multiple cameras and is cleaner to insert.

File: urdf/realsense-RS200.macro.xacro (robot description, xacro)
@@ -1,5 +1,5 @@
 <?xml version="1.0" ?>
 <!--Develped by Daniel Ordonez 22.05.2018 - daniels.ordonez@gmail.com
-    INFORMATIONd:
+    INFORMATION:
         This xacro file a URDF representation of the intel real sense RS200 with the
         virtual links representing the position of:
@@ -11,7 +11,7 @@
 -->
 <robot xmlns:xacro="http://ros.org/wiki/xacro">
-<xacro:macro name="realsense-rs200">
+<xacro:macro name="realsense-rs200" params="prefix parent *origin">
     <!-- Camera link -->
-    <link name="rs200_camera">
+    <link name="${prefix}rs200_camera">
         <visual>
             <origin rpy="0 0 0" xyz="0 0 0"/>
@@ -37,30 +37,36 @@
         </inertial>
     </link>
+    <!-- Connect camera to parent frame-->
+    <joint name="${prefix}realsense_joint" type="fixed">
+        <parent link="${parent}"/>
+        <child link="${prefix}rs200_camera"/>
+        <xacro:insert_block name="origin"/>
+    </joint>
     <!-- Virtual links representing the cameras positons and orientations-->
-    <link name="color" />
-    <link name="depth" />
-    <link name="ired1" />
-    <link name="ired2" />
+    <link name="${prefix}color" />
+    <link name="${prefix}depth" />
+    <link name="${prefix}ired1" />
+    <link name="${prefix}ired2" />
     <!-- Joints positioning the virtual links with respect to the camera main link-->
-    <joint name="color_joint" type="fixed">
-        <parent link="rs200_camera" />
-        <child link="color" />
+    <joint name="${prefix}color_joint" type="fixed">
+        <parent link="${prefix}rs200_camera" />
+        <child link="${prefix}color" />
         <!-- <origin xyz="0 -0.046 0.004" rpy="0 0 0"/> -->
         <!-- The default position is change since in Rviz the cloud depth axis is Z not X-->
         <origin xyz="0 -0.046 0.004" rpy="${pi/2} ${pi} ${pi/2}"/>
     </joint>
-    <joint name="depth_joint" type="fixed">
-        <parent link="rs200_camera" />
-        <child link="depth" />
+    <joint name="${prefix}depth_joint" type="fixed">
+        <parent link="${prefix}rs200_camera" />
+        <child link="${prefix}depth" />
         <origin xyz="0 -0.03 0.004" rpy="0 0 0"/>
     </joint>
-    <joint name="ired1_joint" type="fixed">
-        <parent link="rs200_camera" />
-        <child link="ired1" />
+    <joint name="${prefix}ired1_joint" type="fixed">
+        <parent link="${prefix}rs200_camera" />
+        <child link="${prefix}ired1" />
         <origin xyz="0 -0.06 0.004" rpy="0 0 0"/>
     </joint>
-    <joint name="ired2_joint" type="fixed">
-        <parent link="rs200_camera" />
-        <child link="ired2" />
+    <joint name="${prefix}ired2_joint" type="fixed">
+        <parent link="${prefix}rs200_camera" />
+        <child link="${prefix}ired2" />
         <origin xyz="0 0.01 0.004" rpy="0 0 0"/>
     </joint>
@@ -73,5 +79,5 @@
     </gazebo>
     <!-- Load parameters to model's main link-->
-    <gazebo reference="rs200_camera">
+    <gazebo reference="${prefix}rs200_camera">
         <self_collide>0</self_collide>
         <enable_wind>0</enable_wind>
@@ -89,5 +95,5 @@
         <sensor name="color" type="camera">
             <pose frame="">0 -0.046 0.004 0 0 0</pose>
-            <camera name="__default__">
+            <camera name="${prefix}rs200_camera">
             <horizontal_fov>1.047</horizontal_fov>
             <image>
@@ -112,5 +118,5 @@
         <sensor name="ired1" type="camera">
             <pose frame="">0 -0.06 0.004 0 0 0</pose>
-            <camera name="__default__">
+            <camera name="${prefix}rs200_camera">
             <horizontal_fov>1.047</horizontal_fov>
             <image>
@@ -135,5 +141,5 @@
         <sensor name="ired2" type="camera">
             <pose frame="">0 0.01 0.004 0 0 0</pose>
-            <camera name="__default__">
+            <camera name="${prefix}rs200_camera">
             <horizontal_fov>1.047</horizontal_fov>
             <image>
@@ -158,5 +164,5 @@
         <sensor name="depth" type="depth">
             <pose frame="">0 -0.03 0.004 0 0 0</pose>
-            <camera name="__default__">
+            <camera name="${prefix}rs200_camera">
             <horizontal_fov>1.047</horizontal_fov>
             <image>

Commit message: URDFs edited to handle multi-links. Example added.

File: urdf/realsense-RS200.macro.xacro (robot description, xacro)
@@ -1,5 +1,5 @@
 <?xml version="1.0" ?>
 <!--Develped by Daniel Ordonez 22.05.2018 - daniels.ordonez@gmail.com
-    INFORMATIONd:
+    INFORMATION:
         This xacro file a URDF representation of the intel real sense RS200 with the
         virtual links representing the position of:
@@ -9,7 +9,10 @@
             * Virtual depth coordinate frame
         Configured to work with Gazebo if desired.
+    Update of Maik93: in order to handle camera positions while attaching the Realsense to other links,
+    optional parameters "parent_link, origin_x, origin_y, origin_z" are implemented.
+    See urdf/rs200_simulation_multilink.xacro for details.
 -->
 <robot xmlns:xacro="http://ros.org/wiki/xacro">
-<xacro:macro name="realsense-rs200">
+<xacro:macro name="realsense-rs200" params="parent_link:='rs200_camera' origin_x:=0 origin_y:=0 origin_z:=0">
     <!-- Camera link -->
     <link name="rs200_camera">
@@ -47,5 +50,5 @@
         <child link="color" />
         <!-- <origin xyz="0 -0.046 0.004" rpy="0 0 0"/> -->
-        <!-- The default position is change since in Rviz the cloud depth axis is Z not X-->
+        <!-- The default position is changed since in Rviz the cloud depth axis is Z not X-->
         <origin xyz="0 -0.046 0.004" rpy="${pi/2} ${pi} ${pi/2}"/>
     </joint>
@@ -73,5 +76,5 @@
     </gazebo>
     <!-- Load parameters to model's main link-->
-    <gazebo reference="rs200_camera">
+    <gazebo reference="${parent_link}">
         <self_collide>0</self_collide>
         <enable_wind>0</enable_wind>
@@ -88,5 +91,5 @@
         <min_depth>0</min_depth>-->
         <sensor name="color" type="camera">
-            <pose frame="">0 -0.046 0.004 0 0 0</pose>
+            <pose frame="">${origin_x + 0} ${origin_y - 0.046} ${origin_z + 0.004} 0 0 0</pose>
             <camera name="__default__">
             <horizontal_fov>1.047</horizontal_fov>
@@ -111,5 +114,5 @@
         </sensor>
         <sensor name="ired1" type="camera">
-            <pose frame="">0 -0.06 0.004 0 0 0</pose>
+            <pose frame="">${origin_x + 0} ${origin_y - 0.06} ${origin_z + 0.004} 0 0 0</pose>
             <camera name="__default__">
             <horizontal_fov>1.047</horizontal_fov>
@@ -134,5 +137,5 @@
         </sensor>
         <sensor name="ired2" type="camera">
-            <pose frame="">0 0.01 0.004 0 0 0</pose>
+            <pose frame="">${origin_x + 0} ${origin_y + 0.01} ${origin_z + 0.004} 0 0 0</pose>
             <camera name="__default__">
             <horizontal_fov>1.047</horizontal_fov>
@@ -157,5 +160,5 @@
         </sensor>
         <sensor name="depth" type="depth">
-            <pose frame="">0 -0.03 0.004 0 0 0</pose>
+            <pose frame="">${origin_x + 0} ${origin_y - 0.03} ${origin_z + 0.004} 0 0 0</pose>
             <camera name="__default__">
             <horizontal_fov>1.047</horizontal_fov>

File: urdf/rs200_simulation.xacro (robot description, xacro)
@@ -9,7 +9,8 @@
     <!-- Create camera instance -->
     <xacro:realsense-rs200/>
-    <!-- Gazebo world link required to position the robot with respect to origin-->
+    <!-- Gazebo world link required to position the robot with respect to origin -->
+    <!-- the name "world" is mandatory for Gazebo! -->
     <link name="world"/>
-    <!-- Place camera referenced to world frame-->
+    <!-- Place camera referenced to world frame -->
     <joint name="realsense_joint" type="fixed">
         <parent link="world"/>
